File: hardware/CurrentSensorUSB/CurrentSensorUSB.kicad_pcb (KiCad board)
At the start: 2 copper layers, 7 parts, among them J1 TC2030, P1 USB_C_Plug_USB2.0, U1 ATSAMD21E18A-A, U2 MCP1703Ax-330xxDB

Commit message: not saved
Connections:
- net /VCC_P3V3 renamed +3.3V
- P1 pad A5: unconnected-(P1-CC-PadA5) -> Net-(P1-CC)
- U1 pad 26: unconnected-(U1-~{RESET}-Pad26) -> Net-(U1-~{RESET})
Changed lines of the file:
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@@
 	(net 1 "unconnected-(P1-SHIELD-PadS1)")
 	(net 2 "unconnected-(P1-VCONN-PadB5)")
-	(net 3 "unconnected-(P1-CC-PadA5)")
+	(net 3 "+3.3V")
 	(net 4 "unconnected-(J1-Pad4)")
 	(net 5 "unconnected-(J1-Pad6)")
@@
 	(net 18 "unconnected-(U1-PA10-Pad13)")
 	(net 19 "unconnected-(U1-PA01-Pad2)")
-	(net 20 "unconnected-(U1-~{RESET}-Pad26)")
+	(net 20 "Net-(P1-CC)")
 	(net 21 "unconnected-(U1-PA22-Pad21)")
 	(net 22 "unconnected-(U1-PA11-Pad14)")
@@
 	(net 38 "GND")
 	(net 39 "Net-(D1-VCC)")
-	(net 40 "/VCC_P3V3")
+	(net 40 "Net-(U1-~{RESET})")
 	(net 41 "Net-(D1-I{slash}O1)")
 	(net 42 "Net-(D1-I{slash}O2)")
@@
 			(layers "F.Cu" "F.Mask" "F.Paste")
 			(roundrect_rratio 0.25)
-			(net 40 "/VCC_P3V3")
+			(net 3 "+3.3V")
 			(pintype "passive")
 		)
@@
 			(layers "F.Cu" "F.Mask" "F.Paste")
 			(roundrect_rratio 0.25)
-			(net 40 "/VCC_P3V3")
+			(net 3 "+3.3V")
 			(pinfunction "VDDANA")
 			(pintype "power_in")
@@
 			(layers "F.Cu" "F.Mask" "F.Paste")
 			(roundrect_rratio 0.25)
-			(net 20 "unconnected-(U1-~{RESET}-Pad26)")
+			(net 40 "Net-(U1-~{RESET})")
 			(pinfunction "~{RESET}")
 			(pintype "input")
@@
 			(layers "F.Cu" "F.Mask" "F.Paste")
 			(roundrect_rratio 0.25)
-			(net 40 "/VCC_P3V3")
+			(net 3 "+3.3V")
 			(pinfunction "VDDIN")
 			(pintype "power_in")
@@
 			(size 0.38 1)
 			(layers "F.Cu" "F.Mask" "F.Paste")
-			(net 3 "unconnected-(P1-CC-PadA5)")
+			(net 20 "Net-(P1-CC)")
 			(pinfunction "CC")
 			(pintype "bidirectional")
@@
 			(layers "F.Cu" "F.Mask" "F.Paste")
 			(roundrect_rratio 0.25)
-			(net 40 "/VCC_P3V3")
+			(net 3 "+3.3V")
 			(pinfunction "VO")
 			(pintype "power_out")

Commit message: pcb layout attempt
Parts:
- added C3: 0.1 μF, Capacitor_SMD:C_0603_1608Metric, F.Cu at (61.0, 87.5)
- added C4: C, Capacitor_SMD:C_0603_1608Metric, F.Cu at (61.0, 96.0)
- added C5: 6.8pF, Capacitor_SMD:C_0603_1608Metric, F.Cu at (46.5, 100.0)
- added C6: 6.8pF, Capacitor_SMD:C_0603_1608Metric, F.Cu at (46.8, 96.5)
- added C7: 1 μF, Capacitor_SMD:C_0603_1608Metric, F.Cu at (64.5, 74.5)
- added J2: Screw_Terminal_01x02, TerminalBlock_Phoenix:TerminalBlock_Phoenix_MKDS-1,5-2_1x02_P5.00mm_Horizontal, F.Cu at (86.0, 107.2)
- added PS1: MEE1S0503SC, Converter_DCDC:Converter_DCDC_Murata_MEE1SxxxxSC_THT, F.Cu at (57.9, 110.8)
- added R1: 5.1K, Resistor_SMD:R_0603_1608Metric, F.Cu at (81.5, 69.5)
- added R2: R_Shunt 100, Resistor_SMD:R_Shunt_Ohmite_LVK12, F.Cu at (77.8, 108.4)
- added R3: 4.7 kΩ, Resistor_SMD:R_0603_1608Metric, F.Cu at (61.2, 92.0)
- added R4: 4.7 kΩ, Resistor_SMD:R_0603_1608Metric, F.Cu at (87.0, 84.5)
- added R5: 4.7 kΩ, Resistor_SMD:R_0603_1608Metric, F.Cu at (87.0, 89.5)
- added R6: 4.7 kΩ, Resistor_SMD:R_0603_1608Metric, F.Cu at (45.5, 88.5)
- added R7: R_F 1 kΩ, Resistor_SMD:R_0603_1608Metric, F.Cu at (61.0, 99.5)
- added SW1: SW_Push, Button_Switch_SMD:SW_MEC_5GSH9, F.Cu at (42.0, 71.0)
- added U3: ADS1113IDGS, Package_SO:TSSOP-10_3x3mm_P0.5mm, F.Cu at (87.8, 97.0)
- added U5: ADuM1250, Package_SO:SOIC-8_3.9x4.9mm_P1.27mm, F.Cu at (74.5, 88.0)
- added Y1: 32.768kHz, 7pF, Crystal:Crystal_SMD_0603-4Pin_6.0x3.5mm, F.Cu at (39.5, 98.0)
- moved U1 35.6 mm to (74.5, 76.5)
- moved U2 24.4 mm to (57.0, 67.0)
- moved P1 17.9 mm to (75.2, 65.0)
- moved J1 15.8 mm to (38.4, 87.2), turned to -90 degrees
- moved D1 14.6 mm to (65.5, 66.5)
- moved C2 1.02 mm to (64.5, 81.5)
- moved C1 0.22 mm to (64.5, 78.0)
Connections:
- C1 pad 1: Net-(D1-VCC) -> +5V
- C1 pad 2: GND -> +5V
- C2 pad 2: GND -> +5V
- D1 pad 1: GND -> +5V
- D1 pad 2: Net-(D1-I/O1) -> /USB_DP
- D1 pad 3: Net-(D1-I/O2) -> /USB_DM
- D1 pad 4: Net-(D1-VCC) -> +5V
- J1 pad 1: unconnected-(J1-Pad1) -> /SWDIO
- J1 pad 2: unconnected-(J1-Pad2) -> +5V
- J1 pad 3: unconnected-(J1-Pad3) -> /SWDCLK
- J1 pad 4: unconnected-(J1-Pad4) -> +5V
- J1 pad 5: unconnected-(J1-Pad5) -> /RESET
- J1 pad 6: unconnected-(J1-Pad6) -> +3.3V
- P1 pad A1: GND -> +5V
- P1 pad A12: GND -> +5V
- P1 pad A4: Net-(D1-VCC) -> +5V
- P1 pad A6: Net-(D1-I/O1) -> /USB_DP
- P1 pad A7: Net-(D1-I/O2) -> /USB_DM
- P1 pad A9: Net-(D1-VCC) -> +5V
- P1 pad B1: GND -> +5V
- P1 pad B12: GND -> +5V
- P1 pad B4: Net-(D1-VCC) -> +5V
- P1 pad B9: Net-(D1-VCC) -> +5V
- U1 pad 1: unconnected-(U1-PA00-Pad1) -> /XIN32
- U1 pad 10: GND -> +5V
- U1 pad 2: unconnected-(U1-PA01-Pad2) -> /XOUT32
- U1 pad 21: unconnected-(U1-PA22-Pad21) -> SDA
- U1 pad 22: unconnected-(U1-PA23-Pad22) -> SCL
- U1 pad 23: unconnected-(U1-PA24-Pad23) -> /USB_DP
- U1 pad 24: unconnected-(U1-PA25-Pad24) -> /USB_DM
- U1 pad 26: Net-(U1-~{RESET}) -> /RESET
- U1 pad 28: GND -> +5V
- U1 pad 29: unconnected-(U1-VDDCORE-Pad29) -> Net-(U1-VDDCORE)
- U1 pad 31: unconnected-(U1-PA30-Pad31) -> /SWDIO
- U1 pad 32: unconnected-(U1-PA31-Pad32) -> /SWDCLK
- U2 pad 1: Net-(D1-VCC) -> +5V
- U2 pad 2: GND -> +5V
Routing:
- net +5V: track 0.00 -> 6.44 mm
