File: hardware/CurrentSensorUSB/CurrentSensorUSB.kicad_sch (KiCad schematic)
At the start: 7 parts, among them J1 TC2030, P1 USB_C_Plug_USB2.0, U1 ATSAMD21E18A-A, U2 MCP1703Ax-330xxDB

Commit message: not saved
Parts:
- added C3: 0.1 μF, symbol Device:C
- added C4: C, symbol Device:C
- added J2: Screw_Terminal_01x02, TerminalBlock_Phoenix:TerminalBlock_Phoenix_MKDS-1,5-2_1x02_P5.00mm_Horizontal, symbol Connector:Screw_Terminal_01x02
- added PS1: MEE1S0503SC, Converter_DCDC:Converter_DCDC_Murata_MEE1SxxxxSC_THT, symbol Converter_DCDC:MEE1S0503SC
- added R1: 5.1K, Resistor_SMD:R_0603_1608Metric, symbol Device:R
- added R2: R_Shunt 100, symbol Device:R_Shunt
- added R3, R4, R5, R6: 4.7 kΩ, symbol Device:R
- added R7: R_F 1 kΩ, symbol Device:R
- added SW1: SW_Push, Button_Switch_SMD:SW_MEC_5GSH9, symbol Switch:SW_Push
- added U3: ADS1113IDGS, Package_SO:TSSOP-10_3x3mm_P0.5mm, symbol Analog_ADC:ADS1113IDGS
- added U5: ADuM1250, Package_SO:SOIC-8_3.9x4.9mm_P1.27mm, symbol Isolator:ADuM1250
Connections:
- net GND is gone; now on net +5V: C1.2, C2.2, D1.1 (GND), P1.A1 (GND), P1.A12 (GND), P1.B1 (GND), P1.B12 (GND), U1.10 (GND), U1.28 (GND), U2.2 (GND)
- net +3.3V: now also J1.6, R5.1, R6.1, U5.8 (VDD2)
- net +5V: now reaches C1.1, D1.4 (VCC), P1.A4 (VBUS), P1.A9 (VBUS), P1.B4 (VBUS), P1.B9 (VBUS), U2.1 (VI)
- net +5V: now also J1.2, J1.4, PS1.1 (-Vin), PS1.2 (+Vin), R1.2, SW1.1, U5.5 (GND2)
- net SWDIO: now reaches J1.1
- net SWDCLK: now reaches J1.3
- net RESET: now reaches J1.5
- net RESET: now also U1.26 (~{RESET}), SW1.2
- net at P1.A5 (CC): now also R1.1
- new net: R4.2, U3.9 (SDA), U5.2 (SDA1)
- new net: R3.2, U3.10 (SCL), U5.3 (SCL1)
- new net: R2.2, R7.1
- new net: C4.1, R7.2, U3.4 (AIN0)
- new net 3.3 V ISO: C3.1, PS1.4 (+Vout), R3.1, R4.1, U3.8 (VDD)
- new net GND_ISO: C3.2, C4.2, PS1.3 (-Vout), R2.3, U3.1 (ADDR), U3.3 (GND), U3.5 (AIN1), U5.4 (GND1)
- new net SCL: R5.2, U5.7 (SDA2)
- new net SDA: R6.2, U5.6 (SCL2)
- new net SENS+: J2.1 (Pin_1), R2.1
- new net SENS-: J2.2 (Pin_2), R2.4
Other:
- note added: "External Debugger"
- note added: "Isolated Current Measurement"
- note added: "USB-C Interface"
- moved on the sheet: C1, C2, D1, J1, U1, U2

Commit message: changes in schematic
Parts:
- added C5, C6: 6.8pF, Capacitor_SMD:C_0603_1608Metric, symbol Device:C
- added C7: 1 μF, Capacitor_SMD:C_0603_1608Metric, symbol Device:C
- added Y1: 32.768kHz, 7pF, Crystal:Crystal_SMD_0603-4Pin_6.0x3.5mm, symbol Device:Crystal_GND2
- C3, C4: footprint (none) -> Capacitor_SMD:C_0603_1608Metric
- R2: footprint (none) -> Resistor_SMD:R_Shunt_Ohmite_LVK12
- R3, R4, R5, R6, R7: footprint (none) -> Resistor_SMD:R_0603_1608Metric
Connections:
- net +5V: now also C5.2, C6.2, C7.1, Y1.2
- net SCL: now also U1.22 (PA23)
- net SDA: now also U1.21 (PA22)
- net SWDCLK: now also U1.32 (PA31)
- net SWDIO: now also U1.31 (PA30)
- net USB_DP: now reaches D1.2 (I/O1), P1.A6 (D+)
- net USB_DP: now also U1.23 (PA24)
- net USB_DM: now reaches D1.3 (I/O2), P1.A7 (D-)
- net USB_DM: now also U1.24 (PA25)
- net XIN32: now reaches U1.1 (PA00)
- net XIN32: now also C5.1, Y1.1
- net XOUT32: now reaches U1.2 (PA01)
- net XOUT32: now also C6.1, Y1.3
- net at U1.29 (VDDCORE): now also C7.2
Other:
- note added: "32kHz Crystal"
- moved on the sheet: SW1

Commit message: forgot to save schmatic
Other:
- title: (none) -> USB Current Sensor
Changed lines of the file:
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@@
 	(paper "A4")
 	(title_block
+		(title "USB Current Sensor")
 		(date "2025-05-18")
+		(rev "1.0")
 	)
 	(rectangle
